Commit message: Added working gazebo harmonic simulation along with moveit and rviz

File: src/handy_config/config/handy_description.ros2_control.xacro (robot description, xacro)
@@ -1,10 +1,18 @@
 <?xml version="1.0"?>
 <robot xmlns:xacro="http://www.ros.org/wiki/xacro">
-    <xacro:macro name="handy_description_ros2_control" params="name initial_positions_file">
+    <xacro:macro name="handy_description_ros2_control" params="name initial_positions_file use_sim:=false">
         <xacro:property name="initial_positions" value="${xacro.load_yaml(initial_positions_file)['initial_positions']}"/>
         <ros2_control name="${name}" type="system">
             <hardware>
-                <!-- By default, set up controllers for simulation. This won't work on real hardware -->
-                <plugin>mock_components/GenericSystem</plugin>
+                <xacro:if value="${use_sim}">
+                    <!-- Gazebo Harmonic simulation -->
+                    <plugin>gz_ros2_control/GazeboSimSystem</plugin>
+                </xacro:if>
+                <xacro:unless value="${use_sim}">
+                    <!-- Mock hardware for testing without simulation -->
+                    <plugin>mock_components/GenericSystem</plugin>
+                    <param name="mock_sensor_commands">false</param>
+                    <param name="state_following_offset">0.0</param>
+                </xacro:unless>
             </hardware>
             <joint name="joint1">

File: src/handy_config/config/handy_description.urdf.xacro (robot description, xacro)
@@ -1,9 +1,16 @@
 <?xml version="1.0"?>
 <robot xmlns:xacro="http://www.ros.org/wiki/xacro" name="handy_description">
-    <xacro:arg name="initial_positions_file" default="initial_positions.yaml" />
-    <!-- Import handy_description urdf file -->
-    <xacro:include filename="$(find handy_description)/urdf/handy_description.urdf" />
-    <!-- Import control_xacro -->
-    <xacro:include filename="handy_description.ros2_control.xacro" />
-    <xacro:handy_description_ros2_control name="FakeSystem" initial_positions_file="$(arg initial_positions_file)"/>
+  <!-- Arguments -->
+  <xacro:arg name="initial_positions_file" default="$(find handy_config)/config/initial_positions.yaml"/>
+  <xacro:arg name="use_sim" default="false"/>
+  <!-- Store arg as property for use in macro -->
+  <xacro:property name="use_sim_prop" value="$(arg use_sim)"/>
+  <xacro:include filename="$(find handy_description)/urdf/handy_description.urdf"/>
+  <xacro:include filename="$(find handy_config)/config/handy_description.gazebo.xacro"/>
+  <xacro:include filename="$(find handy_config)/config/handy_description.ros2_control.xacro"/>
+  <!-- Call macro with use_sim property -->
+  <xacro:handy_description_ros2_control
+    name="handy_ros2_control"
+    use_sim="${use_sim_prop}"
+    initial_positions_file="$(arg initial_positions_file)"/>
 </robot>

File: src/handy_description/urdf/handy_description.urdf (robot description, URDF)
Before this commit: robot handy_description, 7 links, 6 joints
Links:
- link Link1: geometry collision mesh filename=file://$(find handy_description)/meshes/Link1.STL; visual mesh filename=file://$(find handy_description)/meshes/Link1.STL
- link Link2: geometry collision mesh filename=file://$(find handy_description)/meshes/Link2.STL; visual mesh filename=file://$(find handy_description)/meshes/Link2.STL
- link Link3: geometry collision mesh filename=file://$(find handy_description)/meshes/Link3.STL; visual mesh filename=file://$(find handy_description)/meshes/Link3.STL
- link Link4: geometry collision mesh filename=file://$(find handy_description)/meshes/Link4.STL; visual mesh filename=file://$(find handy_description)/meshes/Link4.STL
- link Link5: geometry collision mesh filename=file://$(find handy_description)/meshes/Link5.STL; visual mesh filename=file://$(find handy_description)/meshes/Link5.STL
- link Link6: geometry collision mesh filename=file://$(find handy_description)/meshes/Link6.STL; visual mesh filename=file://$(find handy_description)/meshes/Link6.STL
- link base_link: geometry collision mesh filename=file://$(find handy_description)/meshes/base_link.STL; visual mesh filename=file://$(find handy_description)/meshes/base_link.STL
