Commit message: added teleop

File: src/handy_config/config/handy_description.gazebo.xacro (robot description, xacro)
@@ -92,4 +92,13 @@
       </ros>
     </plugin>
+    <plugin name="gz_ros2_control" filename="libgz_ros2_control.so">
+    <ros>
+      <namespace>/</namespace>
+    </ros>
+    <parameters>
+      $(find handy_config)/config/ros2_controllers.yaml
+      $(find handy_config)/config/initial_positions.yaml
+    </parameters>
+  </plugin>
   </gazebo>
 </robot>

File: src/handy_config/config/handy_description.ros2_control.xacro (robot description, xacro)
@@ -12,5 +12,5 @@
                     <!-- Mock hardware for testing without simulation -->
                     <plugin>mock_components/GenericSystem</plugin>
-                    <param name="mock_sensor_commands">false</param>
+                    <param name="mock_sensor_commands">true</param>
                     <param name="state_following_offset">0.0</param>
                 </xacro:unless>
@@ -18,4 +18,5 @@
             <joint name="joint1">
                 <command_interface name="position"/>
+                <command_interface name="velocity"/>
                 <state_interface name="position">
                   <param name="initial_value">${initial_positions['joint1']}</param>
@@ -25,4 +26,5 @@
             <joint name="joint2">
                 <command_interface name="position"/>
+                <command_interface name="velocity"/>
                 <state_interface name="position">
                   <param name="initial_value">${initial_positions['joint2']}</param>
@@ -32,4 +34,5 @@
             <joint name="joint3">
                 <command_interface name="position"/>
+                <command_interface name="velocity"/>
                 <state_interface name="position">
                   <param name="initial_value">${initial_positions['joint3']}</param>
@@ -39,4 +42,5 @@
             <joint name="joint4">
                 <command_interface name="position"/>
+                <command_interface name="velocity"/>
                 <state_interface name="position">
                   <param name="initial_value">${initial_positions['joint4']}</param>
@@ -46,4 +50,5 @@
             <joint name="joint5">
                 <command_interface name="position"/>
+                <command_interface name="velocity"/>
                 <state_interface name="position">
                   <param name="initial_value">${initial_positions['joint5']}</param>
@@ -53,4 +58,5 @@
             <joint name="joint6">
                 <command_interface name="position"/>
+                <command_interface name="velocity"/>
                 <state_interface name="position">
                   <param name="initial_value">${initial_positions['joint6']}</param>

File: src/handy_description/urdf/handy_description.urdf (robot description, URDF)
Before this commit: robot handy_description, 7 links, 6 joints
Joints:
- joint joint1: limit (none) -> lower=-3.14159 upper=3.14159 effort=100 velocity=1.0; type continuous -> revolute
- joint joint2: limit (none) -> lower=-3.14159 upper=3.14159 effort=100 velocity=1.0; type continuous -> revolute
- joint joint3: limit (none) -> lower=-3.14159 upper=3.14159 effort=100 velocity=1.0; type continuous -> revolute
- joint joint4: limit (none) -> lower=-3.14159 upper=3.14159 effort=100 velocity=1.0; type continuous -> revolute
- joint joint5: limit (none) -> lower=-3.14159 upper=3.14159 effort=100 velocity=1.0; type continuous -> revolute
- joint joint6: limit (none) -> lower=-3.14159 upper=3.14159 effort=100 velocity=1.0; type continuous -> revolute

Commit message: added new urdf

File: src/handy_config/config/handy_description.gazebo.xacro (robot description, xacro)
@@ -1,6 +1,5 @@
 <?xml version="1.0"?>
-<!-- filepath: /home/rishik/handy/src/handy_description/urdf/handy_description.gazebo.xacro -->
 <robot xmlns:xacro="http://www.ros.org/wiki/xacro">
-  <!-- Gazebo Colors -->
+  <!-- Gazebo Colors (link names match URDF: Link1, Link2, etc.) -->
   <gazebo reference="base_link">
     <visual>
@@ -12,5 +11,5 @@
     </visual>
   </gazebo>
-  <gazebo reference="link1">
+  <gazebo reference="Link1">
     <visual>
       <material>
@@ -21,5 +20,5 @@
     </visual>
   </gazebo>
-  <gazebo reference="link2">
+  <gazebo reference="Link2">
     <visual>
       <material>
@@ -30,5 +29,5 @@
     </visual>
   </gazebo>
-  <gazebo reference="link3">
+  <gazebo reference="Link3">
     <visual>
       <material>
@@ -39,5 +38,5 @@
     </visual>
   </gazebo>
-  <gazebo reference="link4">
+  <gazebo reference="Link4">
     <visual>
       <material>
@@ -48,5 +47,5 @@
     </visual>
   </gazebo>
-  <gazebo reference="link5">
+  <gazebo reference="Link5">
     <visual>
       <material>
@@ -57,27 +56,9 @@
     </visual>
   </gazebo>
-  <gazebo reference="link6">
+  <gazebo reference="Link6">
     <visual>
       <material>
         <ambient>0.79 0.82 0.93 1</ambient>
         <diffuse>0.79 0.82 0.93 1</diffuse>
-        <specular>0.1 0.1 0.1 1</specular>
-      </material>
-    </visual>
-  </gazebo>
-  <gazebo reference="finger1">
-    <visual>
-      <material>
-        <ambient>0.3 0.3 0.3 1</ambient>
-        <diffuse>0.3 0.3 0.3 1</diffuse>
-        <specular>0.1 0.1 0.1 1</specular>
-      </material>
-    </visual>
-  </gazebo>
-  <gazebo reference="finger2">
-    <visual>
-      <material>
-        <ambient>0.3 0.3 0.3 1</ambient>
-        <diffuse>0.3 0.3 0.3 1</diffuse>
         <specular>0.1 0.1 0.1 1</specular>
       </material>
@@ -92,13 +73,4 @@
       </ros>
     </plugin>
-    <plugin name="gz_ros2_control" filename="libgz_ros2_control.so">
-    <ros>
-      <namespace>/</namespace>
-    </ros>
-    <parameters>
-      $(find handy_config)/config/ros2_controllers.yaml
-      $(find handy_config)/config/initial_positions.yaml
-    </parameters>
-  </plugin>
   </gazebo>
 </robot>

File: src/handy_description/urdf/handy_description.urdf (robot description, URDF)
Before this commit: robot handy_description, 7 links, 6 joints
Links:
- link Link1: mass 1.84719084699337 -> 2.77021151255874
- link Link2: mass 1.79378971577605 -> 1.60258240510756
- link Link3: mass 1.67831155597823 -> 1.41915559432314
- link Link4: mass 0.788294501444391 -> 0.659855119108978
- link Link5: mass 0.666997164681847 -> 0.671110398226165
- link Link6: mass 0.395089923264463 -> 0.372994201208974
- link base_link: mass 5.20579669773012 -> 1.96296034373238
Joints:
- joint joint1: limit lower=-3.14159 upper=3.14159 effort=100 velocity=1.0 -> lower=-3.14159 upper=3.14159 effort=10.0 velocity=1.0; origin xyz=0 0 0.16499999999999 rpy=1.5707963267949 0 -1.78820384774425 -> xyz=0 0 0.203 rpy=1.5707963267949 0 0.90056162865229
- joint joint2: limit lower=-3.14159 upper=3.14159 effort=100 velocity=1.0 -> lower=-3.14159 upper=3.14159 effort=10.0 velocity=1.0; origin xyz=0 0.0980000000000102 0 rpy=0.0331729718675605 0 0 -> xyz=0 0.0980000000000003 0 rpy=-0.845855816973644 0 0
- joint joint3: axis 0 0 1 -> 1 0 0; limit lower=-3.14159 upper=3.14159 effort=100 velocity=1.0 -> lower=-3.14159 upper=3.14159 effort=10.0 velocity=1.0; origin xyz=0 0.29155 0.000575582702538871 rpy=1.5707963267949 -1.32183280290932 1.5707963267949 -> xyz=0 0.28755 0.000575582702541239 rpy=0.94622374788271 0 0
- joint joint4: limit lower=-3.14159 upper=3.14159 effort=100 velocity=1.0 -> lower=-3.14159 upper=3.14159 effort=10.0 velocity=1.0; origin xyz=0 -0.283 0.0937268862500288 rpy=1.5707963267949 0 -2.80898508991109 -> xyz=0 0.25 0 rpy=-3.14159265358979 1.09522041714727 1.5707963267949
- joint joint5: limit lower=-3.14159 upper=3.14159 effort=100 velocity=1.0 -> lower=-3.14159 upper=3.14159 effort=10.0 velocity=1.0; origin xyz=0 0.123067608467674 -0.0836321372682999 rpy=-1.5707963267949 0 -3.07906203524659 -> xyz=0 0.196914494717703 0 rpy=-1.5707963267949 0 -1.36718767182522
- joint joint6: limit lower=-3.14159 upper=3.14159 effort=100 velocity=1.0 -> lower=-3.14159 upper=3.14159 effort=10.0 velocity=1.0; origin xyz=0 0.0921623574494037 -0.0859488892195215 rpy=-1.5707963267949 0 2.60725709980123 -> xyz=0 0.157794494717703 0 rpy=-1.5707963267949 0 2.5989448107597
